File: Carrier_PCB/Carrier_PCB.kicad_sch (KiCad schematic)
At the start: 39 parts, among them J1 Conn_01x24, J2 Conn_01x24

Commit message: Update PCB. Not wired yet
Parts:
- removed C3: 470u, Capacitor_THT:CP_Radial_D10.0mm_P5.00mm, symbol Device:C_Polarized
- removed C5: 100n, Capacitor_SMD:C_0805_2012Metric, symbol Device:C
- added R2: 10K, Resistor_SMD:R_0603_1608Metric, symbol Device:R
- added R3: 20K, Resistor_SMD:R_0603_1608Metric, symbol Device:R
- C1: value 100u -> 10u; footprint Capacitor_THT:CP_Radial_D8.0mm_P3.50mm -> Capacitor_SMD:C_1206_3216Metric
- renumbered C4 to C3
Connections:
- net +3.3V: no longer J_RXSR1.2 (Pin_2), J_RXSR2.2 (Pin_2)
- net +5V: now also C2.2, J_RXSR1.2 (Pin_2), J_RXSR2.2 (Pin_2); no longer C2.1
- net GND: now also C1.2, C2.1, D1.1 (K), R3.2
- net at J2.2 (Pin_2), TP_SBUS1.1: now also J_RXSR1.4 (Pin_4), J_RXSR2.4 (Pin_4)
- net SPORT_MCU: now reaches J2.3 (Pin_3), TP_SPORT1.1
- net SPORT_MCU: now also R2.2, R3.1; no longer J_RXSR1.3 (Pin_3), J_RXSR2.3 (Pin_3)
- new net SPORT_RX: J_RXSR1.3 (Pin_3), J_RXSR2.3 (Pin_3), R2.1
- no-connect marks 0 -> 1
Other:
- moved on the sheet: TP_SBUS1, TP_SPORT1
