File: Carrier_PCB/Carrier_PCB.kicad_pcb (KiCad board)
At the start: 2 copper layers, 99 x 40 mm, 39 parts, among them J1 Conn_01x24, J2 Conn_01x24

Commit message: Update PCB. Not wired yet
Parts:
- J_ESC1: footprint Connector_PinSocket_2.54mm:PinSocket_1x08_P2.54mm_Horizontal -> Connector_PinHeader_2.54mm:PinHeader_1x08_P2.54mm_Horizontal
- J_RXSR1: value Conn_01x05 -> Conn_01x04; footprint Connector_PinSocket_2.54mm:PinSocket_1x05_P2.54mm_Horizontal -> Connector_PinHeader_2.54mm:PinHeader_1x04_P2.54mm_Horizontal
- TP_GND1: value TestPoint -> Conn_01x01; footprint TestPoint:TestPoint_Bridge_Pitch2.54mm_Drill0.7mm -> Connector_PinHeader_2.54mm:PinHeader_1x01_P2.54mm_Horizontal
- moved TP_M1 41.0 mm to (95.0, 133.5)
- moved TP_M2 38.9 mm to (95.0, 129.1)
- moved TP_M3 37.4 mm to (95.0, 124.7)
- moved TP_M4 29.9 mm to (95.2, 104.0)
- moved TP_GND1 23.5 mm to (117.4, 125.8), turned to -90 degrees
- moved J_ESC2 23.3 mm to (93.6, 115.0), turned to -90 degrees
- moved J_ESC1 11.3 mm to (106.3, 103.8), turned to 90 degrees
- moved J_RXSR1 8.52 mm to (167.8, 103.4), turned to 90 degrees
- moved C4 3.93 mm to (104.1, 125.3), turned to -90 degrees
- moved TP_SDI1 3.10 mm to (120.6, 134.0)
- moved TP_SD1 1.90 mm to (123.0, 134.0)
- moved TP_INT1 0.70 mm to (125.4, 133.9)
Connections:
- C1 pad 2: GND -> Net-(D1-K)
- C2 pad 2: GND -> Net-(D1-K)
- D1 pad 1: GND -> Net-(D1-K)

Commit message: Update PCB. Not wired yet
Other:
- board size 99 x 40 mm -> 102.2 x 40 mm
Changed lines of the file:
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@@
 			)
 		)
-		(pad "1" thru_hole rect
+		(pad "1" thru_hole circle
 			(at 0 0 90)
 			(size 1.7 1.7)
@@
 			(pintype "passive")
 		)
-		(pad "2" thru_hole circle
+		(pad "2" thru_hole rect
 			(at 0 2.54 90)
 			(size 1.7 1.7)
@@
 			)
 		)
-		(pad "1" thru_hole rect
+		(pad "1" thru_hole circle
 			(at 0 0 90)
 			(size 1.7 1.7)
@@
 			(pintype "passive")
 		)
-		(pad "6" thru_hole circle
+		(pad "6" thru_hole rect
 			(at 0 12.7 90)
 			(size 1.7 1.7)
@@
 			)
 		)
-		(pad "1" thru_hole rect
+		(pad "1" thru_hole circle
 			(at 0 0 90)
 			(size 1.7 1.7)
@@
 			(pintype "passive")
 		)
-		(pad "23" thru_hole circle
+		(pad "23" thru_hole rect
 			(at 0 55.88 90)
 			(size 1.7 1.7)
@@
 	)
 	(gr_line
-		(start 94 96.25)
-		(end 94 134.25)
+		(start 90.75 109.55)
+		(end 90.8 120.45)
+		(stroke
+			(width 0.05)
+			(type default)
+		)
+		(layer "Edge.Cuts")
+	)
+	(gr_line
+		(start 90.75 109.55)
+		(end 93 109.55)
+		(stroke
+			(width 0.05)
+			(type default)
+		)
+		(layer "Edge.Cuts")
+	)
+	(gr_line
+		(start 90.8 120.45)
+		(end 93 120.45)
+		(stroke
+			(width 0.05)
+			(type default)
+		)
+		(layer "Edge.Cuts")
+	)
+	(gr_arc
+		(start 93 120.45)
+		(mid 93.707107 120.742893)
+		(end 94 121.45)
 		(stroke
 			(width 0.05)
@@
 		(stroke
 			(width 0.05)
+			(type default)
+		)
+		(layer "Edge.Cuts")
+	)
+	(gr_arc
+		(start 94 108.55)
+		(mid 93.707107 109.257107)
+		(end 93 109.55)
+		(stroke
+			(width 0.05)
+			(type default)
+		)
+		(layer "Edge.Cuts")
+	)
+	(gr_line
+		(start 94 108.55)
+		(end 94 96.25)
+		(stroke
+			(width 0.05)
+			(type default)
+		)
+		(layer "Edge.Cuts")
+	)
+	(gr_line
+		(start 94 121.45)
+		(end 94 134.25)
+		(stroke
+			(width 0.05)
