File: Carrier_PCB/Carrier_PCB.kicad_pcb (KiCad board)
At the start: 2 copper layers, 102.2 x 40 mm, 39 parts, among them J1 Conn_01x24, J2 Conn_01x24

Commit message: Update PCB. Not wired yet
Parts:
- removed the C3 at (109.8, 132.4)
- removed C5: 100n, Capacitor_SMD:C_0805_2012Metric
- added R2: 10K, Resistor_SMD:R_0603_1608Metric, F.Cu at (189.5, 116.3)
- added R3: 20K, Resistor_SMD:R_0603_1608Metric, F.Cu at (189.5, 112.7)
- C1: value 100u -> 10u; footprint Capacitor_THT:CP_Radial_D8.0mm_P3.50mm -> Capacitor_SMD:C_1206_3216Metric
- moved C2 58.2 mm to (123.3, 105.9), turned to 0 degrees
- moved GND 46.6 mm to (163.9, 127.0)
- moved TLM1 40.4 mm to (115.7, 133.9)
- moved M4 31.6 mm to (105.5, 133.9)
- moved 3V3 21.6 mm to (157.6, 133.9)
- moved 5V 20.8 mm to (160.3, 133.9)
- moved M1 17.7 mm to (112.7, 133.9)
- moved C1 16.4 mm to (184.1, 119.6), turned to 180 degrees
- moved M2 16.0 mm to (110.2, 133.9)
- moved M3 15.8 mm to (107.8, 133.9)
- moved RXSR 10.1 mm to (172.2, 132.2)
- moved C3 9.74 mm to (98.2, 117.6)
- moved D1 4.11 mm to (137.8, 132.8)
- moved R1 3.10 mm to (136.8, 129.1), turned to -90 degrees
- moved NCS 1.05 mm to (138.6, 99.1)
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- renumbered TP_3V1 to 3V3, TP_5V1 to 5V, C4 to C3, J_ESC1 to ESC1, J_ESC2 to ESC2, TP_GND1 to GND, TP_INT1 to INT, TP_M1 to M1, TP_M2 to M2, TP_M3 to M3, TP_M4 to M4, J_MPU1 to MPU, H_MPU1 to MPU1, H_MPU2 to MPU2, TP_NCS1 to NCS, J_RXSR1 to RXSR, J_RXSR2 to RXSR, TP_SBUS1 to SBUS, TP_SCLK1 to SCLK, TP_SD1 to SD0, TP_SDI1 to SDI, TP_SPORT1 to SPORT, TP_TLM1 to TLM1
Connections:
- C1 pad 2: Net-(D1-K) -> GND
- C2 pad 1: +5V -> GND
- C2 pad 2: Net-(D1-K) -> +5V
- D1 pad 1: Net-(D1-K) -> GND
- J2 pad 3: Net-(J2-Pin_3) -> SPORT_MCU
- RXSR pad 2: +3.3V -> +5V (x2)
- RXSR pad 3: Net-(J2-Pin_3) -> SPORT_RX (x2)
- RXSR pad 4: Net-(J_RXSR1-Pin_4) -> Net-(J2-Pin_2) (x2)
- SPORT pad 1: Net-(J2-Pin_3) -> SPORT_MCU
Routing:
- net GND: track 0.00 -> 213.3 mm, vias 0 -> 6
- net +5V: track 0.00 -> 178.7 mm, vias 0 -> 5
- net Net-(J2-Pin_5): track 0.00 -> 133.6 mm, vias 0 -> 3
- net Net-(J2-Pin_4): track 0.00 -> 132.1 mm, vias 0 -> 3
- net Net-(J2-Pin_6): track 0.00 -> 132.1 mm, vias 0 -> 3
- net Net-(J2-Pin_7): track 0.00 -> 124.1 mm, vias 0 -> 2
- net Net-(J2-Pin_9): track 0.00 -> 123.5 mm, vias 0 -> 2
- net Net-(J1-Pin_11): track 0.00 -> 102.8 mm, vias 0 -> 4
- net +3.3V: track 0.00 -> 90.2 mm, vias 0 -> 1
- net Net-(J2-Pin_13): track 0.00 -> 75.8 mm, vias 0 -> 3
- net Net-(J2-Pin_18): track 0.00 -> 66.1 mm
- net Net-(J2-Pin_14): track 0.00 -> 64.6 mm, vias 0 -> 2
- net Net-(J2-Pin_12): track 0.00 -> 64.5 mm, vias 0 -> 2
- net SPORT_RX: track 0.00 -> 62.7 mm
- net Net-(J2-Pin_2): track 0.00 -> 62.1 mm, vias 0 -> 2
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- added copper zone on B.Cu, net GND
- added copper zone on F.Cu, net GND
Other:
- board size 102.2 x 40 mm -> 102.7 x 40 mm
