File: Carrier_PCB_v2/Carrier_PCB_v2.kicad_pcb (KiCad board)
At the start: 2 copper layers, 102.7 x 40 mm, 39 parts, among them J1 Conn_01x24, J2 Conn_01x24, M1 TestPoint, M2 TestPoint, M3 TestPoint, M4 TestPoint

Commit message: Update PCB. Not wired yet
Parts:
- removed GND: Conn_01x01, Connector_PinHeader_2.54mm:PinHeader_1x01_P2.54mm_Horizontal
- added GND1: 5011, TestPoint:TestPoint_Keystone_5010-5014_Multipurpose, F.Cu at (164.8, 128.0)
- 3V1: renamed from 3V3; value TestPoint -> 5009; footprint TestPoint:TestPoint_Bridge_Pitch2.54mm_Drill0.7mm -> TestPoint:TestPoint_Keystone_5005-5009_Compact
- 5V1: renamed from 5V; value TestPoint -> 5009; footprint TestPoint:TestPoint_Bridge_Pitch2.54mm_Drill0.7mm -> TestPoint:TestPoint_Keystone_5005-5009_Compact
- C1: value 10u -> CL31A106KBHNNNE
- C2, C3: value 100n -> CC0805KRX7R9BB104
- D1: value LED -> NCD0805R1
- ESC1: value Conn_01x08 -> HXPZ2.54-1x8PWZ
- ESC2: value Conn_01x08 -> SM08B-SRSS-TB(LF)(SN)
- INT1: renamed from INT; value TestPoint -> 5009; footprint TestPoint:TestPoint_Bridge_Pitch2.54mm_Drill0.7mm -> TestPoint:TestPoint_Keystone_5005-5009_Compact
- J1, J2: value Conn_01x24 -> HC-PM254-8.5H-1x24PZ
- M1, M2, M3, M4: value TestPoint -> 5009; footprint TestPoint:TestPoint_Bridge_Pitch2.54mm_Drill0.7mm -> TestPoint:TestPoint_Keystone_5005-5009_Compact
- MPU1: renamed from MPU; value Conn_01x10 -> PM2.54-1*10
- NCS1: renamed from NCS; value TestPoint -> 5009; footprint TestPoint:TestPoint_Bridge_Pitch2.54mm_Drill0.7mm -> TestPoint:TestPoint_Keystone_5005-5009_Compact
- R1: value 300 -> 0805W8F3000T5E
- R2: value 10K -> 0603WAF1002T5E
- R3: value 20K -> 0603WAF2002T5E
- RXSR1: renamed from RXSR; value Conn_01x04 -> HC-PZ254-13.8L-1x4PWA
- RXSR2: renamed from RXSR; value Conn_01x04 -> 532610471
- SBUS1: renamed from SBUS; value TestPoint -> 5009; footprint TestPoint:TestPoint_Bridge_Pitch2.54mm_Drill0.7mm -> TestPoint:TestPoint_Keystone_5005-5009_Compact
- SCLK1: renamed from SCLK; value TestPoint -> 5009; footprint TestPoint:TestPoint_Bridge_Pitch2.54mm_Drill0.7mm -> TestPoint:TestPoint_Keystone_5005-5009_Compact
- SDI1: renamed from SDI; value TestPoint -> 5009; footprint TestPoint:TestPoint_Bridge_Pitch2.54mm_Drill0.7mm -> TestPoint:TestPoint_Keystone_5005-5009_Compact
- SDO1: renamed from SD0; value TestPoint -> 5009; footprint TestPoint:TestPoint_Bridge_Pitch2.54mm_Drill0.7mm -> TestPoint:TestPoint_Keystone_5005-5009_Compact
- SPORT1: renamed from SPORT; value TestPoint -> 5009; footprint TestPoint:TestPoint_Bridge_Pitch2.54mm_Drill0.7mm -> TestPoint:TestPoint_Keystone_5005-5009_Compact
- TLM1: renamed from TLM; value TestPoint -> 5009; footprint TestPoint:TestPoint_Bridge_Pitch2.54mm_Drill0.7mm -> TestPoint:TestPoint_Keystone_5005-5009_Compact
- moved SDI1 3.88 mm to (118.8, 130.2)
- moved M1 3.81 mm to (113.5, 130.2)
- moved INT1 3.78 mm to (124.0, 130.2)
- moved M3 3.74 mm to (108.2, 130.2)
- moved NCS1 2.44 mm to (138.8, 101.5)
- moved SBUS1 1.96 mm to (162.4, 98.6)
- moved SCLK1 1.83 mm to (136.2, 97.2)
- moved 5V1 1.61 mm to (161.8, 133.2)
- moved SPORT1 1.59 mm to (157.8, 97.5)
- moved SDO1 1.13 mm to (121.4, 133.2)
- moved M2 0.94 mm to (110.9, 133.2)
- moved TLM1 0.83 mm to (116.1, 133.2)
- moved M4 0.72 mm to (105.7, 133.2)
- moved 3V1 0.72 mm to (157.8, 133.2)
- renumbered MPU1 to H_MPU1, MPU2 to H_MPU2
Routing:
- net Net-(J2-Pin_12): track 64.5 -> 59.6 mm
- net Net-(J2-Pin_2): track 62.1 -> 57.9 mm
- net Net-(J2-Pin_21): track 44.4 -> 40.4 mm
- net Net-(ESC1-Pin_4): track 132.1 -> 128.9 mm
- net Net-(J2-Pin_13): track 75.8 -> 72.7 mm
- net Net-(J2-Pin_14): track 64.6 -> 61.8 mm
- net Net-(ESC1-Pin_3): track 133.6 -> 131.0 mm
- net +5V: track 178.7 -> 176.2 mm
- net Net-(ESC1-Pin_1): track 124.1 -> 121.9 mm
- net SPORT_MCU: track 43.1 -> 42.2 mm
- net Net-(J1-Pin_11): track 102.8 -> 101.9 mm
- net Net-(ESC1-Pin_7): track 123.5 -> 124.3 mm
- net Net-(ESC1-Pin_2): track 132.1 -> 132.7 mm
Other:
- board text added: "DroNyx"
- board text removed: "DRONE PROJECT"
