File: Hardware/ismd_fc_sensortest/ismd_fc_sensortest.kicad_sch (KiCad schematic)
At the start: 11 parts, among them U4 BMI088, U6 ICM-42688-P

Commit message: sensortest chematics
Parts:
- removed C55, C56, C61, C62: 100nF, Capacitor_SMD:C_0402_1005Metric, symbol Device:C
- removed C70: 0.1uF, Capacitor_SMD:C_0402_1005Metric, symbol Device:C
- removed C72: 10nF, Capacitor_SMD:C_0402_1005Metric, symbol Device:C
- removed C74: 2.2uF, Capacitor_SMD:C_0402_1005Metric, symbol Device:C
- removed DPS311: DPS310XTSA1, DPS310XTSA1:XDCR_DPS310XTSA1, symbol DPS310XTSA1:DPS310XTSA1
- removed U4: BMI088, Package_LGA:Bosch_LGA-16_4.5x3mm_P0.5mm_LayoutBorder7x1y_ClockwisePinNumbering, symbol Sensor_Motion:BMI088
- removed U6: ICM-42688-P, ICM-42688-P:PQFN50P300X250X97-14N, symbol ICM-42688-P:ICM-42688-P
- renumbered TEENSY4.2 to U1
Connections:
- net GND: now also U1.45 (GND_1)
- net SCK: now also U1.13 (SCK)
- net SDI: now also U1.11 (MOSI)
- net SDO: now also U1.12 (MISO)
- net INT_B1: now reaches U1.14 (A0)
- net INT_B3: now reaches U1.15 (A1)
- net INT_B5: now reaches U1.16 (A2)
- net INT_I1_1: now reaches U1.17 (A3)
- net INT_I1_2: now reaches U1.18 (A4)
- net INT_I2_1_ACCEL: now reaches U1.19 (A5)
- net INT_I2_2_ACCEL: now reaches U1.20 (A6)
- net INT_I2_3_GYRO: now reaches U1.21 (A7)
- net INT_I2_4_GYRO: now reaches U1.22 (A8)
- net INT_I3_1: now reaches U1.23 (A9)
- net INT_I3_2: now reaches U1.24 (A10)
- net INT_I4_1: now reaches U1.25 (A11)
- net INT_I4_2: now reaches U1.26 (A12)
- net CS_B1: now reaches U1.27 (A13)
- net CS_B2: now reaches U1.28 (RX7)
- net CS_B3: now reaches U1.29 (TX7)
- net CS_B4: now reaches U1.38 (A14)
- net CS_B5: now reaches U1.39 (A15)
- net CS_B6: now reaches U1.40 (A16)
- net CS_I1: now reaches U1.41 (A17)
- net CS_I2_ACCEL: now reaches U1.57 (RX1)
- net +5V renamed +BATT
- net BMP0_INT: no longer names the net of U1.9 (OUT1C)
- net BMP1_INT: no longer names the net of U1.10 (CS_1)
- net BNO_INT renamed CS_I3
- net BNO_RST renamed CS_I2_GYRO
- net L3G_INT1: no longer names the net of U1.8 (TX2)
- net L3G_INT2: no longer names the net of U1.7 (RX2)
- net LSM_INT1: no longer names the net of U1.5 (IN2)
- net LSM_INT2: no longer names the net of U1.4 (BCLK2)
- net LSM_INT3: no longer names the net of U1.6 (OUT1D)
- net MPU_INT renamed CS_I4
- no-connect marks 40 -> 24
Other:
- sheet BMP581 renamed B1-BMP581
- sheet DPS368 renamed B2-DPS368
- added sheet B3-ICP-20100 (b3_icp20100.kicad_sch)
- added sheet B4-MS5611 (b4_msn611.kicad_sch)
- added sheet B5-LPS22DF (b5_lps22df.kicad_sch)
- added sheet B6_ENS220 (b6_ens220.kicad_sch)
- added sheet I1-ICM-42688-P (i1_icm42688p.kicad_sch)
- added sheet I2-BMI088 (i2_bmi088.kicad_sch)
- added sheet I3-BMI270 (i3_bmi270.kicad_sch)
- added sheet I4-ISM330DLC (i4_ism330dlc.kicad_sch)
- sheet B1-BMP581: file bmp581.kicad_sch -> b1_bmp581.kicad_sch
- sheet B2-DPS368: file dps368.kicad_sch -> b2_dps368.kicad_sch
- sheet B2-DPS368 ports: added SCK; removed SDK
- moved on the sheet: U1

Commit message: schematic corrections
Connections:
- net CS_B1: now also U1.39 (A15); no longer U1.27 (A13)
- net CS_B4: now also U1.40 (A16); no longer U1.38 (A14)
- net CS_B5: now also U1.41 (A17); no longer U1.39 (A15)
- net CS_B6: now also U1.1 (TX1); no longer U1.40 (A16)
- net CS_I1: now also U1.2 (OUT2); no longer U1.41 (A17)
- net CS_I2_GYRO: now also U1.3 (LRCLK2); no longer U1.1 (TX1)
- net CS_I3: now also U1.5 (IN2); no longer U1.2 (OUT2)
- net CS_I4: now also U1.6 (OUT1D); no longer U1.3 (LRCLK2)
- net INT_I4_2: now also U1.38 (A14); no longer U1.26 (A12)
- net SDO2: now reaches U1.4 (BCLK2)
- net +BATT renamed +5V
- net SCK renamed SCK1
- net SDI renamed SDI1
- net SDO renamed SDO1
- new net SCK2: U1.27 (A13)
- new net SDI2: U1.26 (A12)
- no-connect marks 24 -> 21
Other:
- removed sheet B6_ENS220

Commit message: sensortest work
Connections:
- net CS_B6: no longer names the net of U1.1 (TX1)
- no-connect marks 21 -> 22
Changed lines of the file:
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@@
+	)
+	(no_connect
+		(at 124.46 33.02)
 	)
 	(no_connect
@@
 		)
 	)
-	(label "CS_B6"
-		(at 124.46 33.02 180)
-		(effects
-			(font
-				(size 1.27 1.27)
-			)
-			(justify right bottom)
-		)
-	)

Commit message: added mounting holes to sensortest
Parts:
- added H1, H10, H2, H3, H4, H5, H6, H7, H8, H9: MountingHole, MountingHole:MountingHole_4mm, symbol Mechanical:MountingHole

Commit message: remove mpu holes in sensortest
Parts:
- removed H10, H9: MountingHole, MountingHole:MountingHole_4mm, symbol Mechanical:MountingHole
- U1: value TEENSY_4.1 -> TEENSY 4.1
Changed lines of the file:
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@@
-	(symbol
-		(lib_id "Mechanical:MountingHole")
-		(at 252.73 76.2 0)
-		(unit 1)
-		(body_style 1)
-		(exclude_from_sim no)
-		(in_bom no)
-		(on_board yes)
-		(in_pos_files yes)
-		(dnp no)
-		(fields_autoplaced yes)
-		(property "Reference" "H9"
-			(at 255.27 74.9299 0)
-			(show_name no)
-			(do_not_autoplace no)
-			(effects
-				(font
-					(size 1.27 1.27)
-				)
-				(justify left)
-			)
-		)
-		(property "Value" "MountingHole"
-			(at 255.27 77.4699 0)
-			(show_name no)
-			(do_not_autoplace no)
-			(effects
-				(font
-					(size 1.27 1.27)
-				)
-				(justify left)
-			)
-		)
-		(property "Footprint" "MountingHole:MountingHole_4mm"
-			(at 252.73 76.2 0)
-			(hide yes)
-			(show_name no)
-			(do_not_autoplace no)
-			(effects
-				(font
-					(size 1.27 1.27)
-				)
-			)
-		)
-		(property "Datasheet" ""
-			(at 252.73 76.2 0)
-			(hide yes)
-			(show_name no)
-			(do_not_autoplace no)
-			(effects
-				(font
-					(size 1.27 1.27)
-				)
-			)
-		)
-		(property "Description" "Mounting Hole without connection"
-			(at 252.73 76.2 0)
-			(hide yes)
-			(show_name no)
-			(do_not_autoplace no)
-			(effects
-				(font
-					(size 1.27 1.27)
-				)
-			)
-		)
-		(instances
-			(project "ismd_fc_sensortest"
-				(path "/ce1b43a9-5bb2-4287-b106-e7fd94ececa3"
-					(reference "H9")
-					(unit 1)
-				)
-			)
-		)
-	)
 	(symbol
 		(lib_id "Mechanical:MountingHole")
@@
 	)
 	(symbol
-		(lib_id "Mechanical:MountingHole")
-		(at 252.73 81.28 0)
-		(unit 1)
-		(body_style 1)
-		(exclude_from_sim no)
-		(in_bom no)
-		(on_board yes)
-		(in_pos_files yes)
-		(dnp no)
-		(fields_autoplaced yes)
-		(property "Reference" "H10"
-			(at 255.27 80.0099 0)
-			(show_name no)
-			(do_not_autoplace no)
-			(effects
-				(font
-					(size 1.27 1.27)
-				)
-				(justify left)
-			)
-		)
-		(property "Value" "MountingHole"
-			(at 255.27 82.5499 0)
-			(show_name no)
-			(do_not_autoplace no)
-			(effects
-				(font
-					(size 1.27 1.27)
-				)
-				(justify left)
-			)
-		)
-		(property "Footprint" "MountingHole:MountingHole_4mm"
-			(at 252.73 81.28 0)
-			(hide yes)
-			(show_name no)
-			(do_not_autoplace no)
-			(effects
-				(font
-					(size 1.27 1.27)
-				)
-			)
-		)
-		(property "Datasheet" ""
-			(at 252.73 81.28 0)
-			(hide yes)
-			(show_name no)
-			(do_not_autoplace no)
-			(effects
-				(font
-					(size 1.27 1.27)
-				)
-			)
-		)
-		(property "Description" "Mounting Hole without connection"
-			(at 252.73 81.28 0)
-			(hide yes)
-			(show_name no)
-			(do_not_autoplace no)
-			(effects
-				(font
-					(size 1.27 1.27)
-				)
-			)
-		)
-		(instances
-			(project "ismd_fc_sensortest"
-				(path "/ce1b43a9-5bb2-4287-b106-e7fd94ececa3"
-					(reference "H10")
-					(unit 1)
-				)
-			)
-		)
-	)
-	(symbol
 		(lib_id "TEENSY_4.1:TEENSY_4.1")
 		(at 124.46 33.02 0)
@@
 			)
 		)
-		(property "Value" "TEENSY_4.1"
+		(property "Value" "TEENSY 4.1"
 			(at 151.13 27.94 0)
 			(show_name no)
