File: Hardware/ismd_fc_sensortest/i4_ism330dlc.kicad_sch (KiCad schematic)
At the start: 3 parts

Commit message: sensortest work
Parts:
- C17: renamed from C20; footprint Capacitor_SMD:C_0402_1005Metric -> Capacitor_SMD:C_0201_0603Metric
- C18: renamed from C19; footprint Capacitor_SMD:C_0402_1005Metric -> Capacitor_SMD:C_0201_0603Metric
- I4: value ISM330DLCTR -> ISM330DLC
Changed lines of the file:
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@@
 		(in_pos_files yes)
 		(dnp no)
-		(property "Reference" "C20"
+		(property "Reference" "C17"
 			(at 68.58 20.066 0)
 			(show_name no)
@@
 			)
 		)
-		(property "Footprint" "Capacitor_SMD:C_0402_1005Metric"
+		(property "Footprint" "Capacitor_SMD:C_0201_0603Metric"
 			(at 63.8048 20.32 0)
 			(hide yes)
@@
 			(project "ismd_fc_sensortest"
 				(path "/ce1b43a9-5bb2-4287-b106-e7fd94ececa3/6e127363-4f9e-4a02-94ac-8294d7e66ed2"
-					(reference "C20")
+					(reference "C17")
 					(unit 1)
 				)
@@
 			)
 		)
-		(property "Value" "ISM330DLCTR"
+		(property "Value" "ISM330DLC"
 			(at 46.99 22.86 0)
 			(show_name no)
@@
 		(in_pos_files yes)
 		(dnp no)
-		(property "Reference" "C19"
+		(property "Reference" "C18"
 			(at 76.454 34.29 0)
 			(show_name no)
@@
 			)
 		)
-		(property "Footprint" "Capacitor_SMD:C_0402_1005Metric"
+		(property "Footprint" "Capacitor_SMD:C_0201_0603Metric"
 			(at 76.2 29.5148 0)
 			(hide yes)
@@
 			(project "ismd_fc_sensortest"
 				(path "/ce1b43a9-5bb2-4287-b106-e7fd94ececa3/6e127363-4f9e-4a02-94ac-8294d7e66ed2"
-					(reference "C19")
+					(reference "C18")
 					(unit 1)
 				)

Commit message: power reg
Parts:
- C17, C18: footprint Capacitor_SMD:C_0201_0603Metric -> Capacitor_SMD:C_0402_1005Metric
Changed lines of the file:
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@@
 			)
 		)
-		(property "Footprint" "Capacitor_SMD:C_0201_0603Metric"
+		(property "Footprint" "Capacitor_SMD:C_0402_1005Metric"
 			(at 63.8048 20.32 0)
 			(hide yes)
@@
 			)
 		)
-		(property "Footprint" "Capacitor_SMD:C_0201_0603Metric"
+		(property "Footprint" "Capacitor_SMD:C_0402_1005Metric"
 			(at 76.2 29.5148 0)
 			(hide yes)
